File: pcb-main2/main2.kicad_pcb (KiCad board)
At the start: 2 copper layers, 113.8 x 59.5 mm, 26 parts, among them U1 ARDUINO_R3_SHIELD_UNO_R3_SHIE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, U2 STM32F103RB, U3 LM2596S_TO263-3, U4 PCF8563, Y1 8MHz

Commit message: finish
Parts:
- moved P-LCD1 34.7 mm to (102.0, 111.8), turned to 90 degrees
- moved P-LCD3 12.0 mm to (83.7, 88.2)
Connections:
- U2 pad 33: Net-(U2-Pad33) -> /D2-A
- U2 pad 34: Net-(U2-Pad34) -> /D2-B
- U2 pad 35: Net-(U2-Pad35) -> /D2-C
- U2 pad 36: Net-(U2-Pad36) -> /D2-D
- U2 pad 37: Net-(U2-Pad37) -> /D1-A
- U2 pad 38: Net-(U2-Pad38) -> /D1-B
- U2 pad 39: Net-(U2-Pad39) -> /D1-C
- U2 pad 40: Net-(U2-Pad40) -> /D1-D
- U2 pad 49: Net-(U2-Pad49) -> /D3-A
- U2 pad 50: Net-(U2-Pad50) -> /D3-B
- U2 pad 51: Net-(U2-Pad51) -> /D3-C
- U2 pad 52: Net-(U2-Pad52) -> /D3-D
Routing:
- net VDD: track 159.0 -> 308.1 mm, vias 7 -> 14
- net /D2-A: track 0.00 -> 131.9 mm, vias 0 -> 1
- net /D2-B: track 0.00 -> 125.9 mm, vias 0 -> 1
- net /D2-C: track 0.00 -> 120.1 mm, vias 0 -> 1
- net /D2-D: track 0.00 -> 114.2 mm, vias 0 -> 1
- net /D3-D: track 0.00 -> 111.9 mm, vias 0 -> 3
- net /D3-C: track 0.00 -> 107.5 mm, vias 0 -> 3
- net /D3-B: track 0.00 -> 101.4 mm, vias 0 -> 3
- net /D3-A: track 0.00 -> 94.4 mm, vias 0 -> 3
- net /LE: track 60.5 -> 150.5 mm, vias 3 -> 5
- net /LD: track 82.2 -> 160.0 mm, vias 3 -> 7
- net /LC: track 79.0 -> 151.5 mm, vias 3 -> 7
- net /D1-D: track 0.00 -> 66.1 mm, vias 0 -> 1
- net /LB: track 76.4 -> 142.5 mm, vias 3 -> 7
- net /D1-C: track 0.00 -> 65.1 mm, vias 0 -> 1
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- added copper zone on B.Cu, net (none)
- added copper zone on F.Cu, net (none)
Other:
- board size 113.8 x 59.5 mm -> 121.3 x 64.1 mm
- net class Default: clearance 0.2 -> 0.15
- rule trace_clearance: 0.2 -> 0.15
