File: pcb-main2/main2.sch (KiCad schematic (older format))
At the start: 26 parts, among them U1 ARDUINO_R3_SHIELD_UNO_R3_SHIE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, U2 STM32F103RB, U3 LM2596S_TO263-3, U4 PCF8563, Y1 8MHz

Commit message: finish
Connections:
- net D1-A: now also U2.37 (PC6)
- net D1-B: now also U2.38 (PC7)
- net D1-C: now also U2.39 (PC8)
- net D1-D: now also U2.40 (PC9)
- net D2-A: now also U2.33 (SPI2_NSS/I2C2_SMBA/USART3_CK/TIM1_BKIN/PB12)
- net D2-B: now also U2.34 (SPI2_SCK/USART3_CTS/TIM1_CH1N/PB13)
- net D2-C: now also U2.35 (SPI2_MISO/USART3_RTS/TIM1_CH2N/PB14)
- net D2-D: now also U2.36 (SPI2_MOSI/TIM1_CH3N/PB15)
- net D3-A: now also U2.49 (JTCK/SWCLK/PA14)
- net D3-B: now also U2.50 (JTDI/PA15)
- net D3-C: now also U2.51 (PC10)
- net D3-D: now also U2.52 (PC11)
Changed lines of the file:
@@
 Text Label 5800 5850 0    60   ~ 0
 LF
+Wire Wire Line
+	5550 6550 5750 6550
+Wire Wire Line
+	5550 6650 5750 6650
+Wire Wire Line
+	5550 6750 5750 6750
+Wire Wire Line
+	5550 6850 5750 6850
+Text Label 5750 6550 0    60   ~ 0
+D2-A
+Text Label 5750 6650 0    60   ~ 0
+D2-B
+Text Label 5750 6750 0    60   ~ 0
+D2-C
+Text Label 5750 6850 0    60   ~ 0
+D2-D
+Wire Wire Line
+	2550 5950 2300 5950
+Wire Wire Line
+	2550 6050 2300 6050
+Wire Wire Line
+	2550 6150 2300 6150
+Wire Wire Line
+	2550 6250 2300 6250
+Text Label 2300 5950 0    60   ~ 0
+D1-A
+Text Label 2300 6050 0    60   ~ 0
+D1-B
+Text Label 2300 6150 0    60   ~ 0
+D1-C
+Text Label 2300 6250 0    60   ~ 0
+D1-D
+Wire Wire Line
+	5550 5050 5800 5050
+Wire Wire Line
+	5550 5150 5800 5150
+Wire Wire Line
+	2300 6350 2550 6350
+Wire Wire Line
+	2550 6450 2300 6450
+Text Label 2300 6350 0    60   ~ 0
+D3-C
+Text Label 2300 6450 0    60   ~ 0
+D3-D
+Text Label 5800 5050 0    60   ~ 0
+D3-A
+Text Label 5800 5150 0    60   ~ 0
+D3-B
 $EndSCHEMATC
